Commit message: Add base_laser to urdf

File: ros/urdf/kagotos1.urdf (robot description, URDF)
Before this commit: robot kagotos1, 3 links, 2 joints
Links:
- added link base_laser; visual cylinder length=0.02 radius=0.03
Joints:
- added joint base_laser_joint: type fixed, parent base_link, child base_laser, origin xyz=0 0 0.08 rpy=0 0 0
